File: SmartSwitch/HW/V1_10312022/1- Design Files/_HW_SmartSwitch/[02] - BLOCK DIAGRAM.kicad_sch (KiCad schematic)
At the start: 0 parts

Commit message: Current and Voltage sampler
Other:
- added sheet PB, RGB ([07]-PB, RGB.kicad_sch)
Changed lines of the file:
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@@
+    )
+  )
+  (sheet (at 161.29 193.04) (size 29.21 27.94) (fields_autoplaced)
+    (stroke (width 0.1524) (type solid) (color 0 0 0 0))
+    (fill (color 0 0 0 0.0000))
+    (property "Sheet name" "PB, RGB" (id 0) (at 161.29 192.3284 0)
+      (effects (font (size 1.27 1.27)) (justify left bottom))
+    )
+    (property "Sheet file" "[07]-PB, RGB.kicad_sch" (id 1) (at 161.29 221.5646 0)
+      (effects (font (size 1.27 1.27)) (justify left top))
     )
   )
