File: SmartSwitch/HW/V1_10312022/1- Design Files/_HW_SmartSwitch/[03] - ESP32, PB.kicad_sch (KiCad schematic)
At the start: 0 parts

Commit message: Current sensor has been done almost :D
Parts:
- added C?: 100nF_16V, Capacitor_SMD:C_0402_1005Metric, symbol SmartSwitch:100nF_16V
- added R? (x2): 10KR_1/20W, Resistor_SMD:R_0201_0603Metric_Pad0.64x0.40mm_HandSolder, symbol SmartSwitch:10KR_1/20W
- added SW?: SPST_NO, symbol SmartSwitch:SPST_NO
Connections:
- new net: C?.2, R?.1, R?.2, SW?.1
- new net +3V3: R?.2
- new net GND: C?.1, SW?.2
- new net PB: R?.1
Changed lines of the file:
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@@
 (kicad_sch (version 20211123) (generator eeschema)
-  (paper "A4")
+  (paper "B")
+  (junction (at 335.28 142.24) (diameter 0) (color 0 0 0 0)
+  )
+  (junction (at 342.9 127) (diameter 0) (color 0 0 0 0)
+  )
+  (junction (at 325.12 127) (diameter 0) (color 0 0 0 0)
+  )
+  (wire (pts (xy 325.12 140.97) (xy 325.12 142.24))
+    (stroke (width 0) (type default) (color 0 0 0 0))
+  )
+  (wire (pts (xy 325.12 127) (xy 325.12 128.27))
+    (stroke (width 0) (type default) (color 0 0 0 0))
+  )
+  (wire (pts (xy 325.12 127) (xy 342.9 127))
+    (stroke (width 0) (type default) (color 0 0 0 0))
+  )
+  (wire (pts (xy 342.9 127) (xy 342.9 128.27))
+    (stroke (width 0) (type default) (color 0 0 0 0))
+  )
+  (wire (pts (xy 342.9 142.24) (xy 342.9 140.97))
+    (stroke (width 0) (type default) (color 0 0 0 0))
+  )
+  (wire (pts (xy 335.28 142.24) (xy 335.28 144.78))
+    (stroke (width 0) (type default) (color 0 0 0 0))
+  )
+  (wire (pts (xy 325.12 142.24) (xy 335.28 142.24))
+    (stroke (width 0) (type default) (color 0 0 0 0))
+  )
+  (wire (pts (xy 335.28 142.24) (xy 342.9 142.24))
+    (stroke (width 0) (type default) (color 0 0 0 0))
+  )
+  (wire (pts (xy 318.77 127) (xy 325.12 127))
+    (stroke (width 0) (type default) (color 0 0 0 0))
+  )
+  (wire (pts (xy 342.9 110.49) (xy 342.9 111.76))
+    (stroke (width 0) (type default) (color 0 0 0 0))
+  )
+  (wire (pts (xy 342.9 124.46) (xy 342.9 127))
+    (stroke (width 0) (type default) (color 0 0 0 0))
+  )
+  (wire (pts (xy 288.29 127) (xy 306.07 127))
+    (stroke (width 0) (type default) (color 0 0 0 0))
+  )
+  (label "PB" (at 288.29 127 0)
+    (effects (font (size 1.27 1.27)) (justify left bottom))
+  )
+  (symbol (lib_id "power:GND") (at 335.28 144.78 0) (unit 1)
+    (in_bom yes) (on_board yes) (fields_autoplaced)
+    (property "Reference" "#PWR?" (id 0) (at 335.28 151.13 0)
+      (effects (font (size 1.27 1.27)) hide)
+    )
+    (property "Value" "GND" (id 1) (at 335.28 149.86 0))
+    (property "Footprint" "" (id 2) (at 335.28 144.78 0)
+      (effects (font (size 1.27 1.27)) hide)
+    )
+    (property "Datasheet" "" (id 3) (at 335.28 144.78 0)
+      (effects (font (size 1.27 1.27)) hide)
+    )
+    (pin "1")
+  )
+  (symbol (lib_id "SmartSwitch:SPST_NO") (at 342.9 128.27 270) (unit 1)
+    (in_bom yes) (on_board yes) (fields_autoplaced)
+    (property "Reference" "SW?" (id 0) (at 346.71 133.2229 90)
+      (effects (font (size 1.27 1.27)) (justify left))
+    )
+    (property "Value" "SPST_NO" (id 1) (at 346.71 135.7629 90)
+      (effects (font (size 1.27 1.27)) (justify left))
+    )
+    (property "Footprint" "" (id 2) (at 342.9 128.27 0)
+      (effects (font (size 1.27 1.27)) hide)
+    )
+    (property "Datasheet" "https://media.digikey.com/pdf/Data%20Sheets/Mitsumi%20Elect/SOU-244HST_7799_ENG_%2317.pdf" (id 3) (at 353.06 176.53 0)
+      (effects (font (size 1.27 1.27)) hide)
+    )
+    (property "Description" "SWITCH TACTILE, SPST-NO, 0.05A 1" (id 4) (at 355.6 144.78 0)
+      (effects (font (size 1.27 1.27)) hide)
+    )
+    (pin "1")
+    (pin "2")
+  )
+  (symbol (lib_id "SmartSwitch:100nF_16V") (at 325.12 140.97 90) (unit 1)
+    (in_bom yes) (on_board yes) (fields_autoplaced)
+    (property "Reference" "C?" (id 0) (at 328.93 133.3499 90)
+      (effects (font (size 1.27 1.27)) (justify right))
+    )
+    (property "Value" "100nF_16V" (id 1) (at 328.93 135.8899 90)
+      (effects (font (size 1.27 1.27)) (justify right))
+    )
+    (property "Footprint" "Capacitor_SMD:C_0402_1005Metric" (id 2) (at 312.42 124.46 0)
+      (effects (font (size 1.27 1.27)) hide)
+    )
+    (property "Datasheet" "https://connect.kemet.com:7667/gateway/IntelliData-ComponentDocumentation/1.0/download/datasheet/C0402C104K4RAC7411" (id 3) (at 309.88 77.47 0)
+      (effects (font (size 1.27 1.27)) hide)
+    )
+    (property "Description" "CAP CER 0.1UF 16V X7R 0402" (id 4) (at 314.96 125.73 0)
+      (effects (font (size 1.27 1.27)) hide)
+    )
+    (pin "1")
+    (pin "2")
+  )
+  (symbol (lib_id "SmartSwitch:10KR_1{slash}20W") (at 306.07 127 0) (unit 1)
+    (in_bom yes) (on_board yes)
+    (property "Reference" "R?" (id 0) (at 320.04 125.73 0))
+    (property "Value" "10KR_1/20W" (id 1) (at 299.72 125.73 0))
+    (property "Footprint" "Resistor_SMD:R_0201_0603Metric_Pad0.64x0.40mm_HandSolder" (id 2) (at 336.55 117.602 0)
+      (effects (font (size 1.27 1.27)) hide)
+    )
+    (property "Datasheet" "https://www.seielect.com/catalog/sei-rmcf_rmcp.pdf" (id 3) (at 332.232 119.888 0)
+      (effects (font (size 1.27 1.27)) hide)
+    )
+    (property "Description" "RES 10K OHM 1% 1/20W 0201" (id 4) (at 321.056 115.316 0)
+      (effects (font (size 1.27 1.27)) hide)
+    )
+    (pin "1")
+    (pin "2")
+  )
+  (symbol (lib_name "10KR_1{slash}20W_1") (lib_id "SmartSwitch:10KR_1{slash}20W") (at 342.9 124.46 90) (unit 1)
+    (in_bom yes) (on_board yes) (fields_autoplaced)
+    (property "Reference" "R?" (id 0) (at 345.44 116.8399 90)
+      (effects (font (size 1.27 1.27)) (justify right))
+    )
+    (property "Value" "10KR_1/20W" (id 1) (at 345.44 119.3799 90)
+      (effects (font (size 1.27 1.27)) (justify right))
+    )
+    (property "Footprint" "Resistor_SMD:R_0201_0603Metric_Pad0.64x0.40mm_HandSolder" (id 2) (at 333.502 93.98 0)
+      (effects (font (size 1.27 1.27)) hide)
+    )
+    (property "Datasheet" "https://www.seielect.com/catalog/sei-rmcf_rmcp.pdf" (id 3) (at 335.788 98.298 0)
+      (effects (font (size 1.27 1.27)) hide)
+    )
+    (property "Description" "RES 10K OHM 1% 1/20W 0201" (id 4) (at 331.216 109.474 0)
+      (effects (font (size 1.27 1.27)) hide)
+    )
+    (pin "1")
+    (pin "2")
+  )
+  (symbol (lib_id "power:+3V3") (at 342.9 110.49 0) (unit 1)
+    (in_bom yes) (on_board yes) (fields_autoplaced)
+    (property "Reference" "#PWR?" (id 0) (at 342.9 114.3 0)
+      (effects (font (size 1.27 1.27)) hide)
+    )
+    (property "Value" "+3V3" (id 1) (at 342.9 105.41 0))
+    (property "Footprint" "" (id 2) (at 342.9 110.49 0)
+      (effects (font (size 1.27 1.27)) hide)
+    )
+    (property "Datasheet" "" (id 3) (at 342.9 110.49 0)
+      (effects (font (size 1.27 1.27)) hide)
+    )
+    (pin "1")
+  )
 )

Commit message: Current and Voltage sampler
Parts:
- removed C?: 100nF_16V, Capacitor_SMD:C_0402_1005Metric, symbol SmartSwitch:100nF_16V
- removed R? (x2): 10KR_1/20W, Resistor_SMD:R_0201_0603Metric_Pad0.64x0.40mm_HandSolder, symbol SmartSwitch:10KR_1/20W
- removed SW?: SPST_NO, symbol SmartSwitch:SPST_NO
Changed lines of the file:
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@@
 (kicad_sch (version 20211123) (generator eeschema)
   (paper "B")
-  (junction (at 335.28 142.24) (diameter 0) (color 0 0 0 0)
-  )
-  (junction (at 342.9 127) (diameter 0) (color 0 0 0 0)
-  )
-  (junction (at 325.12 127) (diameter 0) (color 0 0 0 0)
-  )
-  (wire (pts (xy 325.12 140.97) (xy 325.12 142.24))
-    (stroke (width 0) (type default) (color 0 0 0 0))
-  )
-  (wire (pts (xy 325.12 127) (xy 325.12 128.27))
-    (stroke (width 0) (type default) (color 0 0 0 0))
-  )
-  (wire (pts (xy 325.12 127) (xy 342.9 127))
-    (stroke (width 0) (type default) (color 0 0 0 0))
-  )
-  (wire (pts (xy 342.9 127) (xy 342.9 128.27))
-    (stroke (width 0) (type default) (color 0 0 0 0))
-  )
-  (wire (pts (xy 342.9 142.24) (xy 342.9 140.97))
-    (stroke (width 0) (type default) (color 0 0 0 0))
-  )
-  (wire (pts (xy 335.28 142.24) (xy 335.28 144.78))
-    (stroke (width 0) (type default) (color 0 0 0 0))
-  )
-  (wire (pts (xy 325.12 142.24) (xy 335.28 142.24))
-    (stroke (width 0) (type default) (color 0 0 0 0))
-  )
-  (wire (pts (xy 335.28 142.24) (xy 342.9 142.24))
-    (stroke (width 0) (type default) (color 0 0 0 0))
-  )
-  (wire (pts (xy 318.77 127) (xy 325.12 127))
-    (stroke (width 0) (type default) (color 0 0 0 0))
-  )
-  (wire (pts (xy 342.9 110.49) (xy 342.9 111.76))
-    (stroke (width 0) (type default) (color 0 0 0 0))
-  )
-  (wire (pts (xy 342.9 124.46) (xy 342.9 127))
-    (stroke (width 0) (type default) (color 0 0 0 0))
-  )
-  (wire (pts (xy 288.29 127) (xy 306.07 127))
-    (stroke (width 0) (type default) (color 0 0 0 0))
-  )
-  (label "PB" (at 288.29 127 0)
-    (effects (font (size 1.27 1.27)) (justify left bottom))
-  )
-  (symbol (lib_id "power:GND") (at 335.28 144.78 0) (unit 1)
-    (in_bom yes) (on_board yes) (fields_autoplaced)
-    (property "Reference" "#PWR?" (id 0) (at 335.28 151.13 0)
-      (effects (font (size 1.27 1.27)) hide)
-    )
-    (property "Value" "GND" (id 1) (at 335.28 149.86 0))
-    (property "Footprint" "" (id 2) (at 335.28 144.78 0)
-      (effects (font (size 1.27 1.27)) hide)
-    )
-    (property "Datasheet" "" (id 3) (at 335.28 144.78 0)
-      (effects (font (size 1.27 1.27)) hide)
-    )
-    (pin "1")
-  )
-  (symbol (lib_id "SmartSwitch:SPST_NO") (at 342.9 128.27 270) (unit 1)
-    (in_bom yes) (on_board yes) (fields_autoplaced)
-    (property "Reference" "SW?" (id 0) (at 346.71 133.2229 90)
-      (effects (font (size 1.27 1.27)) (justify left))
-    )
-    (property "Value" "SPST_NO" (id 1) (at 346.71 135.7629 90)
-      (effects (font (size 1.27 1.27)) (justify left))
-    )
-    (property "Footprint" "" (id 2) (at 342.9 128.27 0)
-      (effects (font (size 1.27 1.27)) hide)
-    )
-    (property "Datasheet" "https://media.digikey.com/pdf/Data%20Sheets/Mitsumi%20Elect/SOU-244HST_7799_ENG_%2317.pdf" (id 3) (at 353.06 176.53 0)
-      (effects (font (size 1.27 1.27)) hide)
-    )
-    (property "Description" "SWITCH TACTILE, SPST-NO, 0.05A 1" (id 4) (at 355.6 144.78 0)
-      (effects (font (size 1.27 1.27)) hide)
-    )
-    (pin "1")
-    (pin "2")
-  )
-  (symbol (lib_id "SmartSwitch:100nF_16V") (at 325.12 140.97 90) (unit 1)
-    (in_bom yes) (on_board yes) (fields_autoplaced)
-    (property "Reference" "C?" (id 0) (at 328.93 133.3499 90)
-      (effects (font (size 1.27 1.27)) (justify right))
-    )
-    (property "Value" "100nF_16V" (id 1) (at 328.93 135.8899 90)
-      (effects (font (size 1.27 1.27)) (justify right))
-    )
-    (property "Footprint" "Capacitor_SMD:C_0402_1005Metric" (id 2) (at 312.42 124.46 0)
-      (effects (font (size 1.27 1.27)) hide)
-    )
-    (property "Datasheet" "https://connect.kemet.com:7667/gateway/IntelliData-ComponentDocumentation/1.0/download/datasheet/C0402C104K4RAC7411" (id 3) (at 309.88 77.47 0)
-      (effects (font (size 1.27 1.27)) hide)
-    )
-    (property "Description" "CAP CER 0.1UF 16V X7R 0402" (id 4) (at 314.96 125.73 0)
-      (effects (font (size 1.27 1.27)) hide)
-    )
-    (pin "1")
-    (pin "2")
-  )
-  (symbol (lib_id "SmartSwitch:10KR_1{slash}20W") (at 306.07 127 0) (unit 1)
-    (in_bom yes) (on_board yes)
-    (property "Reference" "R?" (id 0) (at 320.04 125.73 0))
-    (property "Value" "10KR_1/20W" (id 1) (at 299.72 125.73 0))
-    (property "Footprint" "Resistor_SMD:R_0201_0603Metric_Pad0.64x0.40mm_HandSolder" (id 2) (at 336.55 117.602 0)
-      (effects (font (size 1.27 1.27)) hide)
-    )
-    (property "Datasheet" "https://www.seielect.com/catalog/sei-rmcf_rmcp.pdf" (id 3) (at 332.232 119.888 0)
-      (effects (font (size 1.27 1.27)) hide)
-    )
-    (property "Description" "RES 10K OHM 1% 1/20W 0201" (id 4) (at 321.056 115.316 0)
-      (effects (font (size 1.27 1.27)) hide)
-    )
-    (pin "1")
-    (pin "2")
-  )
-  (symbol (lib_name "10KR_1{slash}20W_1") (lib_id "SmartSwitch:10KR_1{slash}20W") (at 342.9 124.46 90) (unit 1)
-    (in_bom yes) (on_board yes) (fields_autoplaced)
-    (property "Reference" "R?" (id 0) (at 345.44 116.8399 90)
-      (effects (font (size 1.27 1.27)) (justify right))
-    )
-    (property "Value" "10KR_1/20W" (id 1) (at 345.44 119.3799 90)
-      (effects (font (size 1.27 1.27)) (justify right))
-    )
-    (property "Footprint" "Resistor_SMD:R_0201_0603Metric_Pad0.64x0.40mm_HandSolder" (id 2) (at 333.502 93.98 0)
-      (effects (font (size 1.27 1.27)) hide)
-    )
-    (property "Datasheet" "https://www.seielect.com/catalog/sei-rmcf_rmcp.pdf" (id 3) (at 335.788 98.298 0)
-      (effects (font (size 1.27 1.27)) hide)
-    )
-    (property "Description" "RES 10K OHM 1% 1/20W 0201" (id 4) (at 331.216 109.474 0)
-      (effects (font (size 1.27 1.27)) hide)
-    )
-    (pin "1")
-    (pin "2")
-  )
-  (symbol (lib_id "power:+3V3") (at 342.9 110.49 0) (unit 1)
-    (in_bom yes) (on_board yes) (fields_autoplaced)
-    (property "Reference" "#PWR?" (id 0) (at 342.9 114.3 0)
-      (effects (font (size 1.27 1.27)) hide)
-    )
-    (property "Value" "+3V3" (id 1) (at 342.9 105.41 0))
-    (property "Footprint" "" (id 2) (at 342.9 110.49 0)
-      (effects (font (size 1.27 1.27)) hide)
-    )
-    (property "Datasheet" "" (id 3) (at 342.9 110.49 0)
-      (effects (font (size 1.27 1.27)) hide)
-    )
-    (pin "1")
-  )
 )
